File: _autosave-BLEANT.sch (KiCad schematic (older format))
At the start: 53 parts, among them IC1 FAN4010IL6X_F113, IC2 FAN4010IL6X_F113, J1 Conn_01x04_Male, J2 SC_19-20, J3 Conn_01x02, J4 Conn_01x02, J5 1909763-1, U1 nRF51x22-QFxx, U2 LM50BIM3, U3 MP5077GG-Z, U4 MP5077GG-Z, X2 32.768kHz, Y1 16MHz

Commit message: Added BOM
Parts:
- C21: value 0.56uF -> 0.68uF
Changed lines of the file:
@@
 P 7450 3200
 F 0 "C21" V 7198 3200 50  0000 C CNN
-F 1 "0.56uF" V 7289 3200 50  0000 C CNN
+F 1 "0.68uF" V 7289 3200 50  0000 C CNN
 F 2 "Capacitor_SMD:C_0402_1005Metric" H 7488 3050 50  0001 C CNN
 F 3 "~" H 7450 3200 50  0001 C CNN
