File: BLEANT.sch (KiCad schematic (older format))
At the start: 62 parts, among them IC1 FAN4010IL6X_F113, IC2 FAN4010IL6X_F113, J1 Conn_01x04_Male, J2 SC_19-20, J3 Conn_01x02, J4 Conn_01x02, J5 1909763-1, U1 nRF51x22-QFxx, U3 MP5077GG-Z, U4 MP5077GG-Z, X2 32.768kHz, Y1 16MHz

Commit message: Added a metric ton of test points
Parts:
- removed R17: 3.3k, Resistor_SMD:R_0402_1005Metric, symbol Device:R_US
- added TP1, TP10, TP11, TP14, TP15, TP2, TP3, TP4, TP5, TP6, TP7, TP8, TP9: 5029, digikey-footprints:PC_Test_Point_Mini_3.8x2.03mm, symbol dk_Test-Points:5029
- added TP16, TP17, TP18: TestPoint, TestPoint:TestPoint_Pad_2.0x2.0mm, symbol Connector:TestPoint
- C21: value 0.68uF -> 47nF
- C22: value 1uF -> 47nF
Connections:
- net +3V3: now also TP9.1
- net +5V: now also TP7.1
- net 3V3Sense: now also TP5.1
- net 5V0Sense: now also TP6.1
- net GND: now also TP8.1
- net MISO: now also TP18.1
- net MOSI: now also TP17.1
- net SCK: now also TP16.1
- net Temperature: now also TP11.1
- net UART_RX: now also TP15.1
- net UART_TX: now also TP14.1
- net at C19.1, IC2.1 (VIN), L7.2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: now also TP3.1
- net at C18.1, D3.1 (A1), J3.1 (Pin_1)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: now also TP1.1
- net at C15.1, D2.1 (A1), J4.1 (Pin_1)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: now also TP2.1
- net at C16.1, IC1.1 (VIN), L9.2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: now also TP4.1
- net at C33.1, C34.1, L6.1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: now also TP10.1
Other:
- note added: "CAN Sheet\n"
- note added: "Power Conditioning\n"
- note added: "Stack Connector\n"
- note added: "Temp Sensor\n"
- note added: "nRF51422"
- moved on the sheet: R8, R9

Commit message: Added some filters and stuff
Parts:
- added C40, C41, C42, C43: 100pF, Capacitor_SMD:C_0402_1005Metric, symbol Device:C
- added R16: 470, Resistor_SMD:R_0402_1005Metric, symbol Device:R_US
Connections:
- net GND: now also C40.2, C41.2, C42.2, C43.2
- net MISO: now also C42.1
- net MOSI: now also C41.1
- net SCK: now also C43.1
- net UART_RX: now also R16.1; no longer U1.47 (P0.28)
- new net: C40.1, R16.2, U1.47 (P0.28)
Changed lines of the file:
@@
 	0    1    1    0
 $EndComp
-Text GLabel 13700 4950 0    50   Input ~ 0
-MOSI
 Text GLabel 13700 5100 0    50   Output ~ 0
 MISO
@@
 Text GLabel 13300 3350 0    50   Output ~ 0
 UART_RX
-Text GLabel 4900 5800 2    50   Input ~ 0
+Text GLabel 5600 5800 2    50   Input ~ 0
 UART_RX
 Text GLabel 4900 5900 2    50   Output ~ 0
@@
 	-1   0    0    1
 $EndComp
+$Comp
+L Device:R_US R16
+U 1 1 5E2CB1E4
+P 5400 5800
+F 0 "R16" V 5195 5800 50  0000 C CNN
+F 1 "470" V 5286 5800 50  0000 C CNN
+F 2 "Resistor_SMD:R_0402_1005Metric" V 5440 5790 50  0001 C CNN
+F 3 "~" H 5400 5800 50  0001 C CNN
+	1    5400 5800
+	0    1    1    0
+$EndComp
+$Comp
+L Device:C C40
+U 1 1 5E2CB56E
+P 5250 5600
+F 0 "C40" H 5135 5554 50  0000 R CNN
+F 1 "100pF" H 5135 5645 50  0000 R CNN
+F 2 "Capacitor_SMD:C_0402_1005Metric" H 5288 5450 50  0001 C CNN
+F 3 "~" H 5250 5600 50  0001 C CNN
+	1    5250 5600
+	-1   0    0    1
+$EndComp
+Wire Wire Line
+	4900 5800 5250 5800
+Wire Wire Line
+	5250 5800 5250 5750
+Connection ~ 5250 5800
+Wire Wire Line
+	5550 5800 5600 5800
+$Comp
+L power:GND #PWR028
+U 1 1 5E2D36FA
+P 5250 5450
+F 0 "#PWR028" H 5250 5200 50  0001 C CNN
+F 1 "GND" H 5255 5277 50  0000 C CNN
+F 2 "" H 5250 5450 50  0001 C CNN
+F 3 "" H 5250 5450 50  0001 C CNN
+	1    5250 5450
+	-1   0    0    1
+$EndComp
+$Comp
+L Device:C C41
+U 1 1 5E2E439D
+P 11300 4350
+F 0 "C41" H 11415 4396 50  0000 L CNN
+F 1 "100pF" H 11415 4305 50  0000 L CNN
+F 2 "Capacitor_SMD:C_0402_1005Metric" H 11338 4200 50  0001 C CNN
+F 3 "~" H 11300 4350 50  0001 C CNN
+	1    11300 4350
+	1    0    0    -1
+$EndComp
+Text GLabel 13700 4950 0    50   Input ~ 0
+MOSI
+Text GLabel 11300 4200 1    50   Input ~ 0
+MOSI
+Text GLabel 11700 4200 1    50   Output ~ 0
+MISO
+Text GLabel 12100 4200 1    50   Input ~ 0
+SCK
+$Comp
+L Device:C C42
+U 1 1 5E2EAF9D
+P 11700 4350
+F 0 "C42" H 11815 4396 50  0000 L CNN
+F 1 "100pF" H 11815 4305 50  0000 L CNN
+F 2 "Capacitor_SMD:C_0402_1005Metric" H 11738 4200 50  0001 C CNN
+F 3 "~" H 11700 4350 50  0001 C CNN
+	1    11700 4350
+	1    0    0    -1
+$EndComp
+$Comp
+L Device:C C43
+U 1 1 5E2EB2C5
+P 12100 4350
+F 0 "C43" H 12215 4396 50  0000 L CNN
+F 1 "100pF" H 12215 4305 50  0000 L CNN
+F 2 "Capacitor_SMD:C_0402_1005Metric" H 12138 4200 50  0001 C CNN
+F 3 "~" H 12100 4350 50  0001 C CNN
+	1    12100 4350
+	1    0    0    -1
+$EndComp
+$Comp
+L power:GND #PWR033
+U 1 1 5E2EBBC7
+P 11300 4500
+F 0 "#PWR033" H 11300 4250 50  0001 C CNN
+F 1 "GND" H 11305 4327 50  0000 C CNN
+F 2 "" H 11300 4500 50  0001 C CNN
+F 3 "" H 11300 4500 50  0001 C CNN
+	1    11300 4500
+	1    0    0    -1
+$EndComp
+$Comp
+L power:GND #PWR034
+U 1 1 5E2EBFE7
+P 11700 4500
+F 0 "#PWR034" H 11700 4250 50  0001 C CNN
+F 1 "GND" H 11705 4327 50  0000 C CNN
+F 2 "" H 11700 4500 50  0001 C CNN
+F 3 "" H 11700 4500 50  0001 C CNN
+	1    11700 4500
+	1    0    0    -1
+$EndComp
+$Comp
+L power:GND #PWR035
+U 1 1 5E2EC191
+P 12100 4500
+F 0 "#PWR035" H 12100 4250 50  0001 C CNN
+F 1 "GND" H 12105 4327 50  0000 C CNN
+F 2 "" H 12100 4500 50  0001 C CNN
+F 3 "" H 12100 4500 50  0001 C CNN
+	1    12100 4500
+	1    0    0    -1
+$EndComp
 $EndSCHEMATC

Commit message: Fixed RF traces
Parts:
- removed J1: Conn_01x04_Male, Connector_PinHeader_2.54mm:PinHeader_1x04_P2.54mm_Vertical, symbol Connector:Conn_01x04_Male
- added J1: SWD, 2X10_BOXHEADER, symbol SWD:SWD
- C1, C10, C11, C12, C13, C14, C15, C16, C18, C19, C2, C21, C22, C3, C31, C32, C33, C34, C35, C36, C4, C40, C41, C42, C43, C5, C6, C7, C8, C9: symbol Device:C -> BLEANT-rescue:C-Device
- D2, D3: symbol Device:D_TVS -> BLEANT-rescue:D_TVS-Device
- IC1, IC2: symbol FAN4010IL6X_F113:FAN4010IL6X_F113 -> BLEANT-rescue:FAN4010IL6X_F113-FAN4010IL6X_F113
- J2: symbol MASA_Library:SC_19-20 -> BLEANT-rescue:SC_19-20-MASA_Library
- J3, J4: symbol Connector_Generic:Conn_01x02 -> BLEANT-rescue:Conn_01x02-Connector_Generic
- J5: symbol 1909763-1:1909763-1 -> BLEANT-rescue:1909763-1-1909763-1
- L1, L2, L3, L4, L5, L6, L7, L9: symbol Device:L -> BLEANT-rescue:L-Device
- R1, R14, R15, R16, R18, R2, R3, R4, R5, R6, R7, R8, R9: symbol Device:R_US -> BLEANT-rescue:R_US-Device
- TMP1: symbol MASA_Library:LM50CIM3X -> BLEANT-rescue:LM50CIM3X-MASA_Library
- TP1, TP10, TP11, TP14, TP15, TP2, TP3, TP4, TP5, TP6, TP7, TP8, TP9: symbol dk_Test-Points:5029 -> BLEANT-rescue:5029-dk_Test-Points
- TP16, TP17, TP18: symbol Connector:TestPoint -> BLEANT-rescue:TestPoint-Connector
- U1: symbol MCU_Nordic:nRF51x22-QFxx -> BLEANT-rescue:nRF51x22-QFxx-MCU_Nordic
- U3, U4: symbol MASA_Library:MP5077GG-Z -> BLEANT-rescue:MP5077GG-Z-MASA_Library
- X2: symbol Device:Crystal -> BLEANT-rescue:Crystal-Device
- Y1: symbol Device:Crystal_GND24 -> BLEANT-rescue:Crystal_GND24-Device
Connections:
- net +3V3: now also J1.1 (VDD)
- net GND: now also J1.3 (GND), J1.5 (GND@1), J1.9 (GND_DETECT)
- net SWDCLK: now also J1.4 (SWDCLK)
- net SWDIO: now also J1.2 (SWDIO)
