File: CAN_Template.sch (KiCad schematic (older format))
At the start: 27 parts, among them U2 SN74LVC1T45DBVR, U5 MCP2515-xSO, U6 SN65HVD1050D, U7 SN74LVC1T45DBVR

Commit message: Fixed RF traces
Parts:
- C17, C20, C23, C24, C25, C26, C27, C28, C29, C30, C37, C38, C39: symbol Device:C -> BLEANT-rescue:C-Device
- D1: symbol Device:D_TVS_x2_CAA -> BLEANT-rescue:D_TVS_x2_CAA-Device
- NP1, NP2, R10, R11, R12, R13, R17: symbol Device:R_US -> BLEANT-rescue:R_US-Device
- TP12, TP13: symbol dk_Test-Points:5029 -> BLEANT-rescue:5029-dk_Test-Points
- U2, U7: symbol dk_Logic-Translators-Level-Shifters:SN74LVC1T45DBVR -> BLEANT-rescue:SN74LVC1T45DBVR-dk_Logic-Translators-Level-Shifters
- U5: symbol Interface_CAN_LIN:MCP2515-xSO -> BLEANT-rescue:MCP2515-xSO-Interface_CAN_LIN
- U6: symbol Interface_CAN_LIN:SN65HVD1050D -> BLEANT-rescue:SN65HVD1050D-Interface_CAN_LIN
Changed lines of the file:
@@
 EESchema Schematic File Version 4
-LIBS:BLEANT-cache
 EELAYER 30 0
 EELAYER END
@@
 CAN_Transciever
 $Comp
-L Device:R_US NP1
+L BLEANT-rescue:R_US-Device NP1
 U 1 1 5DCB3E43
 P 7950 3250
@@
 $EndComp
 $Comp
-L Device:C C25
+L BLEANT-rescue:C-Device C25
 U 1 1 5DCB9CD1
 P 7100 2700
@@
 $EndComp
 $Comp
-L Device:C C26
+L BLEANT-rescue:C-Device C26
 U 1 1 5DCBAD85
 P 7100 2900
@@
 $EndComp
 $Comp
-L power:GND #PWR09
+L BLEANT-rescue:GND-power #PWR09
 U 1 1 5DCE500D
 P 1450 3050
@@
 $EndComp
 $Comp
-L Device:C C28
+L BLEANT-rescue:C-Device C28
 U 1 1 5DCE6703
 P 7950 4150
@@
 $EndComp
 $Comp
-L Device:R_US NP2
+L BLEANT-rescue:R_US-Device NP2
 U 1 1 5DCE98D1
 P 7950 3650
@@
 $EndComp
 $Comp
-L Device:C C29
+L BLEANT-rescue:C-Device C29
 U 1 1 5DCEFDFD
 P 8250 3450
@@
 $EndComp
 $Comp
-L power:GND #PWR019
+L BLEANT-rescue:GND-power #PWR019
 U 1 1 5DCF0F65
 P 7950 4300
@@
 $EndComp
 $Comp
-L power:GND #PWR018
+L BLEANT-rescue:GND-power #PWR018
 U 1 1 5DCF11EA
 P 7950 2600
@@
 $EndComp
 $Comp
-L Device:R_US R13
+L BLEANT-rescue:R_US-Device R13
 U 1 1 5DCF1CE0
 P 7650 3450
@@
 $EndComp
 $Comp
-L Device:D_TVS_x2_CAA D1
+L BLEANT-rescue:D_TVS_x2_CAA-Device D1
 U 1 1 5DD0169A
 P 8700 3450
@@
 $EndComp
 $Comp
-L Device:R_US R12
+L BLEANT-rescue:R_US-Device R12
 U 1 1 5DD5BD7B
 P 6200 3900
@@
 $EndComp
 $Comp
-L Device:R_US R11
+L BLEANT-rescue:R_US-Device R11
 U 1 1 5DD67335
 P 2550 3350
@@
 $EndComp
 $Comp
-L Interface_CAN_LIN:MCP2515-xSO U5
+L BLEANT-rescue:MCP2515-xSO-Interface_CAN_LIN U5
 U 1 1 5DCB05B0
 P 1450 3850
@@
 CAN_H
 $Comp
-L Device:C C27
+L BLEANT-rescue:C-Device C27
 U 1 1 5DCE5998
 P 7950 2750
@@
 $EndComp
 $Comp
-L Interface_CAN_LIN:SN65HVD1050D U6
+L BLEANT-rescue:SN65HVD1050D-Interface_CAN_LIN U6
 U 1 1 5DD4ABBA
 P 6800 3450
@@
 Connection ~ 8700 3000
 $Comp
-L power:GND #PWR015
+L BLEANT-rescue:GND-power #PWR015
 U 1 1 5E09CBC9
 P 6800 3850
@@
 $EndComp
 $Comp
-L power:GND #PWR017
+L BLEANT-rescue:GND-power #PWR017
 U 1 1 5E0A1057
 P 7250 2900
@@
 $EndComp
 $Comp
-L power:GND #PWR016
+L BLEANT-rescue:GND-power #PWR016
 U 1 1 5E0A1679
 P 7250 2700
@@
 Connection ~ 6800 2900
 $Comp
-L power:+5V #PWR014
+L BLEANT-rescue:+5V-power #PWR014
 U 1 1 5E0A2EDD
 P 6800 2700
@@
 	6200 3650 6300 3650
 $Comp
-L power:GND #PWR013
+L BLEANT-rescue:GND-power #PWR013
 U 1 1 5E0A7026
 P 6200 4050
@@
 $EndComp
 $Comp
-L Device:R_US R10
+L BLEANT-rescue:R_US-Device R10
 U 1 1 5E0A7D89
 P 5950 3250
@@
 $EndComp
 $Comp
-L Device:C C20
+L BLEANT-rescue:C-Device C20
 U 1 1 5E0BDAE5
 P 1150 5000
@@
 $EndComp
 $Comp
-L Device:C C17
+L BLEANT-rescue:C-Device C17
 U 1 1 5E0BDAEB
 P 1150 4800
@@
 $EndComp
 $Comp
-L power:GND #PWR07
+L BLEANT-rescue:GND-power #PWR07
 U 1 1 5E0BDAF1
 P 1000 4800
@@
 $EndComp
 $Comp
-L power:GND #PWR08
+L BLEANT-rescue:GND-power #PWR08
 U 1 1 5E0BDAF7
 P 1000 5000
@@
 Connection ~ 1450 4800
 $Comp
-L Device:C C24
+L BLEANT-rescue:C-Device C24
 U 1 1 5E0C191D
 P 2700 3750
@@
 $EndComp
 $Comp
-L power:GND #PWR012
+L BLEANT-rescue:GND-power #PWR012
 U 1 1 5E0C3AF0
 P 2700 3900
@@
 	8400 3450 8450 3450
 $Comp
-L power:GND #PWR020
+L BLEANT-rescue:GND-power #PWR020
 U 1 1 5E0C862A
 P 8450 3450
@@
 	6250 3350 6300 3350
 $Comp
-L power:+3V3 #PWR010
+L BLEANT-rescue:+3V3-power #PWR010
 U 1 1 5E0C8133
 P 1450 5300
@@
 	5650 3100 5650 3250
 $Comp
-L power:GND #PWR011
+L BLEANT-rescue:GND-power #PWR011
 U 1 1 5E0B3A8E
 P 5650 2800
@@
 $EndComp
 $Comp
-L Device:C C23
+L BLEANT-rescue:C-Device C23
 U 1 1 5DCB7D7B
 P 5650 2950
@@
 CAN Controller
 $Comp
-L Device:R_US R17
+L BLEANT-rescue:R_US-Device R17
 U 1 1 5E27A6F5
 P 1450 5150
@@
 $EndComp
 $Comp
-L dk_Test-Points:5029 TP12
+L BLEANT-rescue:5029-dk_Test-Points TP12
 U 1 1 5E2BCF1F
 P 8700 2900
@@
 $EndComp
 $Comp
-L dk_Test-Points:5029 TP13
+L BLEANT-rescue:5029-dk_Test-Points TP13
 U 1 1 5E2BE1B4
 P 8700 4000
@@
 $EndComp
 $Comp
-L power:GND #PWR0140
+L BLEANT-rescue:GND-power #PWR0140
 U 1 1 5E2BB7E8
 P 4250 3100
@@
 $EndComp
 $Comp
-L power:+5V #PWR0141
+L BLEANT-rescue:+5V-power #PWR0141
 U 1 1 5E2BB304
 P 4250 2150
@@
 $EndComp
 $Comp
-L power:+3V3 #PWR0142
+L BLEANT-rescue:+3V3-power #PWR0142
 U 1 1 5E2BAB74
 P 4150 2150
@@
 $EndComp
 $Comp
-L dk_Logic-Translators-Level-Shifters:SN74LVC1T45DBVR U2
+L BLEANT-rescue:SN74LVC1T45DBVR-dk_Logic-Translators-Level-Shifters U2
 U 1 1 5E2B9A42
 P 4150 2700
@@
 	5450 2700 5450 3250
 $Comp
-L power:GND #PWR0143
+L BLEANT-rescue:GND-power #PWR0143
 U 1 1 5E2CAD52
 P 4250 4400
@@
 $EndComp
 $Comp
-L power:+5V #PWR0144
+L BLEANT-rescue:+5V-power #PWR0144
 U 1 1 5E2CAD58
 P 4250 3500
@@
 $EndComp
 $Comp
-L power:+3V3 #PWR0145
+L BLEANT-rescue:+3V3-power #PWR0145
 U 1 1 5E2CAD5E
 P 4150 3500
@@
 $EndComp
 $Comp
-L dk_Logic-Translators-Level-Shifters:SN74LVC1T45DBVR U7
+L BLEANT-rescue:SN74LVC1T45DBVR-dk_Logic-Translators-Level-Shifters U7
 U 1 1 5E2CAD6D
 P 4150 4000
@@
 	5450 4000 5450 3350
 $Comp
-L power:GND #PWR0146
+L BLEANT-rescue:GND-power #PWR0146
 U 1 1 5E2CE665
 P 3850 2900
@@
 $EndComp
 $Comp
-L power:+3V3 #PWR0147
+L BLEANT-rescue:+3V3-power #PWR0147
 U 1 1 5E2CEA35
 P 3850 4200
@@
 $EndComp
 $Comp
-L Device:C C37
+L BLEANT-rescue:C-Device C37
 U 1 1 5E2F2DDF
 P 3950 2200
@@
 $EndComp
 $Comp
-L Device:C C38
+L BLEANT-rescue:C-Device C38
 U 1 1 5E2B9A2B
 P 4450 2200
@@
 	4150 2200 4150 2300
 $Comp
-L power:GND #PWR025
+L BLEANT-rescue:GND-power #PWR025
 U 1 1 5E2BEEB8
 P 3800 2200
@@
 $EndComp
 $Comp
-L power:GND #PWR026
+L BLEANT-rescue:GND-power #PWR026
 U 1 1 5E2BF3E6
 P 4600 2200
@@
 $EndComp
 $Comp
-L Device:C C39
+L BLEANT-rescue:C-Device C39
 U 1 1 5E2BF78D
 P 4500 3600
@@
 $EndComp
 $Comp
-L Device:C C30
+L BLEANT-rescue:C-Device C30
 U 1 1 5E2C02EF
 P 3850 3600
@@
 Connection ~ 4150 3600
 $Comp
-L power:GND #PWR024
+L BLEANT-rescue:GND-power #PWR024
 U 1 1 5E2C6515
 P 3700 3600
@@
 $EndComp
 $Comp
-L power:GND #PWR027
+L BLEANT-rescue:GND-power #PWR027
 U 1 1 5E2C6B9B
 P 4650 3600
